File: Schematics/Section A - Title A.kicad_sch (KiCad schematic)
At the start: 0 parts

Commit message: Update Template
Other:
- note added: "Rakesh Bhanavath"
- note removed: "J. Pieper ADC investigation"
Changed lines of the file:
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@@
 		)
 	)
-	(text "J. Pieper ADC investigation"
+	(text "Rakesh Bhanavath"
 		(exclude_from_sim no)
 		(at 142.24 170.18 0)
@@
 			)
 			(justify left bottom)
-			(href "https://jpieper.com/2023/07/24/stm32g4-adc-performance-part-2/")
+			(href "https://github.com/rakeshbhanavath")
 		)
 	)
