File: Schematics/USB.kicad_sch (KiCad schematic)
At the start: 7 parts, among them J1201 USB_C_Receptacle_USB2.0_16P

Commit message: WIP
Parts:
- removed D1005, D1006: BPESD0402-05ST, Diode_SMD:D_0402_1005Metric, symbol Device:D_TVS
- added U2: USBLC6-2P6, EasyEDA:SOT-666-6_L1.6-W1.2-P0.50-LS1.6-BL, symbol Power_Protection:USBLC6-2P6
Connections:
- net GND: now also U2.2 (GND)
- net USB_ESD_D+: now also U2.1 (I/O1); no longer R1203.1
- net USB_ESD_D-: now also U2.3 (I/O2); no longer R1204.1
- net VBUS: now also U2.5 (VBUS)
- new net USB_R_D+: R1203.1, U2.6 (I/O1)
- new net USB_R_D-: R1204.1, U2.4 (I/O2)
